Commit message: URDF - added power bank and fix laser x offset

File: description/gazebo_control.xacro (robot description, xacro)
@@ -6,6 +6,6 @@
             <left_joint>left_wheel_joint</left_joint>
             <right_joint>right_wheel_joint</right_joint>
-            <wheel_separation>0.3</wheel_separation>
-            <wheel_diameter>0.1</wheel_diameter>
+            <wheel_separation>0.199</wheel_separation>
+            <wheel_diameter>0.065</wheel_diameter>
             <!-- Limits -->
             <max_wheel_torque>200.0</max_wheel_torque>

File: description/lidar.xacro (robot description, xacro)
@@ -1,5 +1,5 @@
 <?xml version="1.0"?>
 <robot xmlns:xacro="http://www.ros.org/wiki/xacro">
-    <xacro:property name="laser_offset_x" value="0"/>
+    <xacro:property name="laser_offset_x" value="0.005"/>
     <xacro:property name="laser_radius" value="0.035"/>
     <xacro:property name="laser_thickness" value="0.02"/>
@@ -13,5 +13,5 @@
         <parent link="chassis"/>
         <child link="laser_base"/>
-        <origin xyz="${laser_base_length/2 - laser_radius} 0 ${chassis_height/2 + laser_base_height/2}" rpy="0 0 0"/>
+        <origin xyz="${laser_base_length/2 - laser_radius - laser_offset_x} 0 ${chassis_height/2 + laser_base_height/2}" rpy="0 0 0"/>
     </joint>
     <link name="laser_base">
@@ -37,5 +37,5 @@
         <parent link="chassis" />
         <child link="laser_frame" />
-        <origin xyz="0 0 ${chassis_height/2 + laser_base_height + laser_thickness/2}" rpy="0 0 0" />
+        <origin xyz="${-laser_offset_x} 0 ${chassis_height/2 + laser_base_height + laser_thickness/2}" rpy="0 0 0" />
     </joint>
     <link name="laser_frame">

File: description/robot_core.xacro (robot description, xacro)
@@ -13,5 +13,5 @@
     <xacro:property name="motor_offset_y" value="0.055"/>
     <xacro:property name="motor_offset_z" value="0.0"/>
-    <xacro:property name="wheel_radius" value="0.0339"/>
+    <xacro:property name="wheel_radius" value="0.0325"/>
     <xacro:property name="wheel_thickness" value="0.025"/>
     <xacro:property name="wheel_mass" value="0.05"/>
@@ -26,4 +26,11 @@
     <xacro:property name="battery_height" value="0.034"/>
     <xacro:property name="battery_mass" value="0.233"/>
+    <xacro:property name="power_bank_length" value="0.105"/>
+    <xacro:property name="power_bank_width" value="0.065"/>
+    <xacro:property name="power_bank_height" value="0.013"/>
+    <xacro:property name="power_bank_mass" value="0.200"/>
+    <xacro:property name="power_bank_offset_x" value="0.09"/>
+    <xacro:property name="power_bank_offset_y" value="0.0"/>
+    <!-- <xacro:property name="power_bank_offset_z" value="0.0"/> -->
     <!-- Define colors -->
     <material name="white">
@@ -284,7 +291,8 @@
     <!-- LIPO BATTERY LINK -->
     <joint name="lipo_battery_joint" type="fixed">
-        <parent link="base_footprint"/>
+        <parent link="chassis"/>
         <child link="lipo_battery"/>
-        <origin xyz="0 0 ${chassis_offset_z - battery_height / 2}" rpy="0 0 0"/>
+        <origin xyz="0 0 ${-chassis_height/2 - battery_height / 2}" rpy="0 0 0"/>
+        <!-- <origin xyz="0 0 ${chassis_offset_z - battery_height / 2}" rpy="0 0 0"/> -->
     </joint>
     <link name="lipo_battery">
@@ -307,3 +315,28 @@
         <material>Gazebo/White</material>
     </gazebo>
+    <!-- POWER BANK LINK -->
+    <joint name="power_bank_joint" type="fixed">
+        <parent link="chassis"/>
+        <child link="power_bank"/>
+        <origin xyz="${power_bank_offset_x} 0 ${chassis_height/2 + power_bank_height/2}" rpy="0 0 ${-pi/2}"/>
+    </joint>
+    <link name="power_bank">
+        <visual>
+            <geometry>
+                <box size="${power_bank_length} ${power_bank_width} ${power_bank_height}"/>
+            </geometry>
+            <material name="white"/>
+        </visual>
+        <collision>
+            <geometry>
+                <box size="${power_bank_length} ${power_bank_width} ${power_bank_height}"/>
+            </geometry>
+        </collision>
+        <xacro:inertial_box mass="${power_bank_mass}" x="${power_bank_length}" y="${power_bank_width}" z="${power_bank_height}">
+            <origin xyz="0 0 0" rpy="0 0 0"/>
+        </xacro:inertial_box>
+    </link>
+    <gazebo reference="power_bank">
+        <material>Gazebo/White</material>
+    </gazebo>
 </robot>
