Commit message: Add robo simulation

File: description/robot_core.xacro (robot description, xacro)
@@ -40,4 +40,7 @@
         </xacro:inertial_box>
     </link>
+    <gazebo reference="chassis">
+        <material>Gazebo/White</material>
+    </gazebo>
     <!-- LEFT WHEEL LINK -->
     <joint name="left_wheel_joint" type="continuous">
@@ -63,4 +66,7 @@
         </xacro:inertial_cylinder>
     </link>
+    <gazebo reference="left_wheel">
+        <material>Gazebo/Blue</material>
+    </gazebo>
     <!-- RIGHT WHEEL LINK -->
     <joint name="right_wheel_joint" type="continuous">
@@ -86,4 +92,7 @@
         </xacro:inertial_cylinder>
     </link>
+    <gazebo reference="right_wheel">
+        <material>Gazebo/Blue</material>
+    </gazebo>
     <!-- FRONT CASTER WHEEL LINK -->
     <joint name="front_caster_joint" type="fixed">
@@ -108,4 +117,9 @@
         </xacro:inertial_sphere>
     </link>
+    <gazebo reference="front_caster_wheel">
+        <material>Gazebo/Black</material>
+        <mu1 value="0.001" />
+        <mu2 value="0.001" />
+    </gazebo>
     <!-- REAR CASTER WHEEL LINK -->
     <joint name="rear_caster_joint" type="fixed">
@@ -130,3 +144,8 @@
         </xacro:inertial_sphere>
     </link>
+    <gazebo reference="rear_caster_wheel">
+        <material>Gazebo/Black</material>
+        <mu1 value="0.001" />
+        <mu2 value="0.001" />
+    </gazebo>
 </robot>

Commit message: Updated URDF with robot diamension

File: description/robot_core.xacro (robot description, xacro)
@@ -2,4 +2,28 @@
 <robot xmlns:xacro="http://www.ros.org/wiki/xacro">
     <xacro:include filename="inertial_macros.xacro" />
+    <xacro:property name="chassis_length" value="0.255"/>
+    <xacro:property name="chassis_width" value="0.15"/>
+    <xacro:property name="chassis_height" value="0.034"/>
+    <xacro:property name="chassis_mass" value="0.5"/>
+    <xacro:property name="chassis_offset_z" value="0.044"/> <!-- Height of the chassis above the ground or base footprint -->
+    <xacro:property name="motor_radius" value="0.01"/>
+    <xacro:property name="motor_thickness" value="0.06"/>
+    <xacro:property name="motor_mass" value="0.08"/>
+    <xacro:property name="motor_offset_x" value="0.0"/>
+    <xacro:property name="motor_offset_y" value="0.055"/>
+    <xacro:property name="motor_offset_z" value="0.0"/>
+    <xacro:property name="wheel_radius" value="0.0339"/>
+    <xacro:property name="wheel_thickness" value="0.025"/>
+    <xacro:property name="wheel_mass" value="0.05"/>
+    <xacro:property name="wheel_offset_x" value="0.0"/>
+    <xacro:property name="wheel_offset_y" value="0.0995"/>
+    <xacro:property name="wheel_offset_z" value="0.0"/>
+    <xacro:property name="caster_wheel_radius" value="0.0065"/>
+    <xacro:property name="caster_wheel_mass" value="0.02"/>
+    <xacro:property name="caster_wheel_offset_x" value="0.098"/>
+    <xacro:property name="battery_length" value="0.112"/>
+    <xacro:property name="battery_width" value="0.032"/>
+    <xacro:property name="battery_height" value="0.034"/>
+    <xacro:property name="battery_mass" value="0.233"/>
     <!-- Define colors -->
     <material name="white">
@@ -15,30 +39,64 @@
         <color rgba="0 0 0 1"/>
     </material>
+    <material name="red">
+        <color rgba="1 0 0 1"/>
+    </material>
+    <!-- BASE_FOOTPRINT LINK -->
+    <link name="base_footprint"></link>
     <!-- BASE LINK -->
+    <joint name="base_link_joint" type="fixed">
+        <parent link="base_footprint"/>
+        <child link="base_link"/>
+        <origin xyz="0 0 ${wheel_radius}" rpy="0 0 0"/>
+    </joint>
     <link name="base_link"></link>
-    <!-- BASE FOOTPRINT LINK -->
     <!-- CHASSIS LINK -->
     <joint name="chassis_joint" type="fixed">
+        <parent link="base_footprint"/>
+        <child link="chassis"/>
+        <origin xyz="0 0 ${chassis_offset_z + chassis_height / 2}" rpy="0 0 0"/>
+    </joint>
+    <link name="chassis">
+        <visual>
+            <geometry>
+                <box size="${chassis_length} ${chassis_width} ${chassis_height}"/>
+            </geometry>
+            <material name="orange"/>
+        </visual>
+        <collision>
+            <geometry>
+                <box size="${chassis_length} ${chassis_width} ${chassis_height}"/>
+            </geometry>
+        </collision>
+        <xacro:inertial_box mass="${chassis_mass}" x="${chassis_length}" y="${chassis_width}" z="${chassis_height}">
+            <origin xyz="0 0 0" rpy="0 0 0"/>
+        </xacro:inertial_box>
+    </link>
+    <gazebo reference="chassis">
+        <material>Gazebo/Orange</material>
+    </gazebo>
+    <!-- LEFT MOTOR LINK -->
+    <joint name="left_motor_joint" type="fixed">
         <parent link="base_link"/>
-        <child link="chassis"/>
-        <origin xyz="0 0 0.1" rpy="0 0 0"/>
-    </joint>
-    <link name="chassis">
-        <visual>
-            <geometry>
-                <box size="0.4 0.3 0.15"/>
-            </geometry>
-            <material name="white"/>
-        </visual>
-        <collision>
-            <geometry>
-                <box size="0.4 0.3 0.15"/>
-            </geometry>
-        </collision>
-        <xacro:inertial_box mass="0.5" x="0.4" y="0.3" z="0.15">
-            <origin xyz="0 0 0" rpy="0 0 0"/>
-        </xacro:inertial_box>
-    </link>
-    <gazebo reference="chassis">
+        <child link="left_motor"/>
+        <origin xyz="0 ${motor_offset_y} 0" rpy="${-pi/2} 0 0" />
+    </joint>
+    <link name="left_motor">
+        <visual>
+            <geometry>
+                <cylinder radius="${motor_radius}" length="${motor_thickness}"/>
+            </geometry>
+            <material name="white"/>
+        </visual>
+        <collision>
+            <geometry>
+                <cylinder radius="${motor_radius}" length="${motor_thickness}"/>
+            </geometry>
+        </collision>
+        <xacro:inertial_cylinder mass="${motor_mass}" length="${motor_thickness}" radius="${motor_radius}">
+            <origin xyz="0 0 0" rpy="0 0 0"/>
+        </xacro:inertial_cylinder>
+    </link>
+    <gazebo reference="left_motor">
         <material>Gazebo/White</material>
     </gazebo>
@@ -47,5 +105,5 @@
         <parent link="base_link"/>
         <child link="left_wheel"/>
-        <origin xyz="0 0.15 0" rpy="-${pi/2} 0 0"/>
+        <origin xyz="0 ${wheel_offset_y} 0" rpy="${-pi/2} 0 0" />
         <axis xyz="0 0 1"/>
     </joint>
@@ -53,5 +111,5 @@
         <visual>
             <geometry>
-                <cylinder radius="0.05" length="0.04"/>
+                <cylinder radius="${wheel_radius}" length="${wheel_thickness}"/>
             </geometry>
             <material name="blue"/>
@@ -59,8 +117,8 @@
         <collision>
             <geometry>
-                <cylinder radius="0.05" length="0.04"/>
-            </geometry>
-        </collision>
-        <xacro:inertial_cylinder mass="0.1" length="0.04" radius="0.05">
+                <sphere radius="${wheel_radius}"/>
+            </geometry>
+        </collision>
+        <xacro:inertial_cylinder mass="${wheel_mass}" length="${wheel_thickness}" radius="${wheel_radius}">
             <origin xyz="0 0 0" rpy="0 0 0"/>
         </xacro:inertial_cylinder>
@@ -68,4 +126,29 @@
     <gazebo reference="left_wheel">
         <material>Gazebo/Blue</material>
+    </gazebo>
+    <!-- RIGHT MOTOR LINK -->
+    <joint name="right_motor_joint" type="fixed">
+        <parent link="base_link"/>
+        <child link="right_motor"/>
+        <origin xyz="0 ${-motor_offset_y} 0" rpy="${pi/2} 0 0" />
+    </joint>
+    <link name="right_motor">
+        <visual>
+            <geometry>
+                <cylinder radius="${motor_radius}" length="${motor_thickness}"/>
+            </geometry>
+            <material name="white"/>
+        </visual>
+        <collision>
+            <geometry>
+                <cylinder radius="${motor_radius}" length="${motor_thickness}"/>
+            </geometry>
+        </collision>
+        <xacro:inertial_cylinder mass="${motor_mass}" length="${motor_thickness}" radius="${motor_radius}">
+            <origin xyz="0 0 0" rpy="0 0 0"/>
+        </xacro:inertial_cylinder>
+    </link>
+    <gazebo reference="right_motor">
+        <material>Gazebo/White</material>
     </gazebo>
     <!-- RIGHT WHEEL LINK -->
@@ -73,5 +156,5 @@
         <parent link="base_link"/>
         <child link="right_wheel"/>
-        <origin xyz="0 -0.15 0" rpy="${pi/2} 0 0"/>
+        <origin xyz="0 ${-wheel_offset_y} 0" rpy="${pi/2} 0 0" />
         <axis xyz="0 0 -1"/>
     </joint>
@@ -79,5 +162,5 @@
         <visual>
             <geometry>
-                <cylinder radius="0.05" length="0.04"/>
+                <cylinder radius="${wheel_radius}" length="${wheel_thickness}"/>
             </geometry>
             <material name="blue"/>
@@ -85,8 +168,8 @@
         <collision>
             <geometry>
-                <cylinder radius="0.05" length="0.04"/>
-            </geometry>
-        </collision>
-        <xacro:inertial_cylinder mass="0.1" length="0.04" radius="0.05">
+                <sphere radius="${wheel_radius}"/>
+            </geometry>
+        </collision>
+        <xacro:inertial_cylinder mass="${wheel_mass}" length="${wheel_thickness}" radius="${wheel_radius}">
             <origin xyz="0 0 0" rpy="0 0 0"/>
         </xacro:inertial_cylinder>
@@ -95,14 +178,39 @@
         <material>Gazebo/Blue</material>
     </gazebo>
+    <!-- FRONT CASTER WHEEL BASE LINK -->
+    <joint name="front_caster_wheel_base_joint" type="fixed">
+        <parent link="base_footprint"/>
+        <child link="front_caster_wheel_base"/>
+        <origin xyz="${caster_wheel_offset_x} 0 ${chassis_offset_z/2 + caster_wheel_radius/2}"/> <!-- front_caster_wheel_base = chassis_offset_z - caster_wheel_radius -->
+    </joint>
+    <link name="front_caster_wheel_base">
+        <visual>
+            <geometry>
+                <cylinder radius="${caster_wheel_radius * 3}" length="${chassis_offset_z - caster_wheel_radius}"/>
+            </geometry>
+            <material name="white"/>
+        </visual>
+        <collision>
+            <geometry>
+                <cylinder radius="${caster_wheel_radius * 3}" length="${chassis_offset_z - caster_wheel_radius}"/>
+            </geometry>
+        </collision>
+        <xacro:inertial_cylinder mass="0.005" length="${chassis_offset_z - caster_wheel_radius}" radius="${caster_wheel_radius * 3}">
+            <origin xyz="0 0 0" rpy="0 0 0"/>
+        </xacro:inertial_cylinder>
+    </link>
+    <gazebo reference="front_caster_wheel_base">
+        <material>Gazebo/White</material>
+    </gazebo>
     <!-- FRONT CASTER WHEEL LINK -->
     <joint name="front_caster_joint" type="fixed">
-        <parent link="base_link"/>
+        <parent link="base_footprint"/>
         <child link="front_caster_wheel"/>
-        <origin xyz="0.15 0 0" rpy="0 0 0"/>
+        <origin xyz="${caster_wheel_offset_x} 0 ${caster_wheel_radius}" rpy="0 0 0"/>
     </joint>
     <link name="front_caster_wheel">
         <visual>
             <geometry>
-                <sphere radius="0.05"/>
+                <sphere radius="${caster_wheel_radius}"/>
             </geometry>
             <material name="black"/>
@@ -110,8 +218,8 @@
         <collision>
             <geometry>
-                <sphere radius="0.05"/>
-            </geometry>
-        </collision>
-        <xacro:inertial_sphere mass="0.05" radius="0.05">
+                <sphere radius="${caster_wheel_radius}"/>
+            </geometry>
+        </collision>
+        <xacro:inertial_sphere mass="${caster_wheel_mass}" radius="${caster_wheel_radius}">
             <origin xyz="0 0 0" rpy="0 0 0"/>
         </xacro:inertial_sphere>
@@ -122,14 +230,39 @@
         <mu2 value="0.001" />
     </gazebo>
+    <!-- REAR CASTER BASE WHEEL LINK -->
+    <joint name="rear_caster_wheel_base_joint" type="fixed">
+        <parent link="base_footprint"/>
+        <child link="rear_caster_wheel_base"/>
+        <origin xyz="${-caster_wheel_offset_x} 0 ${chassis_offset_z/2 + caster_wheel_radius/2}"/> <!-- rear_caster_wheel_base = chassis_offset_z - caster_wheel_radius -->
+    </joint>
+    <link name="rear_caster_wheel_base">
+        <visual>
+            <geometry>
+                <cylinder radius="${caster_wheel_radius * 3}" length="${chassis_offset_z - caster_wheel_radius}"/>
+            </geometry>
+            <material name="white"/>
+        </visual>
+        <collision>
+            <geometry>
+                <cylinder radius="${caster_wheel_radius * 3}" length="${chassis_offset_z - caster_wheel_radius}"/>
+            </geometry>
+        </collision>
+        <xacro:inertial_cylinder mass="0.005" length="${chassis_offset_z - caster_wheel_radius}" radius="${caster_wheel_radius * 3}">
+            <origin xyz="0 0 0" rpy="0 0 0"/>
+        </xacro:inertial_cylinder>
+    </link>
+    <gazebo reference="rear_caster_wheel_base">
+        <material>Gazebo/White</material>
+    </gazebo>
     <!-- REAR CASTER WHEEL LINK -->
     <joint name="rear_caster_joint" type="fixed">
-        <parent link="base_link"/>
+        <parent link="base_footprint"/>
         <child link="rear_caster_wheel"/>
-        <origin xyz="-0.15 0 0" rpy="0 0 0"/>
+        <origin xyz="${-caster_wheel_offset_x} 0 ${caster_wheel_radius}" rpy="0 0 0"/>
     </joint>
     <link name="rear_caster_wheel">
         <visual>
             <geometry>
-                <sphere radius="0.05"/>
+                <sphere radius="${caster_wheel_radius}"/>
             </geometry>
             <material name="black"/>
@@ -137,8 +270,8 @@
         <collision>
             <geometry>
-                <sphere radius="0.05"/>
-            </geometry>
-        </collision>
-        <xacro:inertial_sphere mass="0.05" radius="0.05">
+                <sphere radius="${caster_wheel_radius}"/>
+            </geometry>
+        </collision>
+        <xacro:inertial_sphere mass="${caster_wheel_mass}" radius="${caster_wheel_radius}">
             <origin xyz="0 0 0" rpy="0 0 0"/>
         </xacro:inertial_sphere>
@@ -149,3 +282,28 @@
         <mu2 value="0.001" />
     </gazebo>
+    <!-- LIPO BATTERY LINK -->
+    <joint name="lipo_battery_joint" type="fixed">
+        <parent link="base_footprint"/>
+        <child link="lipo_battery"/>
+        <origin xyz="0 0 ${chassis_offset_z - battery_height / 2}" rpy="0 0 0"/>
+    </joint>
+    <link name="lipo_battery">
+        <visual>
+            <geometry>
+                <box size="${battery_length} ${battery_width} ${battery_height}"/>
+            </geometry>
+            <material name="white"/>
+        </visual>
+        <collision>
+            <geometry>
+                <box size="${battery_length} ${battery_width} ${battery_height}"/>
+            </geometry>
+        </collision>
+        <xacro:inertial_box mass="${battery_mass}" x="${battery_length}" y="${battery_width}" z="${battery_height}">
+            <origin xyz="0 0 0" rpy="0 0 0"/>
+        </xacro:inertial_box>
+    </link>
+    <gazebo reference="lipo_battery">
+        <material>Gazebo/White</material>
+    </gazebo>
 </robot>

Commit message: odom parameter tuning for better accuracy

File: description/robot_core.xacro (robot description, xacro)
@@ -15,7 +15,7 @@
     <xacro:property name="wheel_radius" value="0.0325"/>
     <xacro:property name="wheel_thickness" value="0.025"/>
-    <xacro:property name="wheel_mass" value="0.05"/>
+    <xacro:property name="wheel_mass" value="0.03"/>
     <xacro:property name="wheel_offset_x" value="0.0"/>
-    <xacro:property name="wheel_offset_y" value="0.0995"/>
+    <xacro:property name="wheel_offset_y" value="0.093"/>
     <xacro:property name="wheel_offset_z" value="0.0"/>
     <xacro:property name="caster_wheel_radius" value="0.0065"/>
@@ -32,5 +32,4 @@
     <xacro:property name="power_bank_offset_x" value="0.09"/>
     <xacro:property name="power_bank_offset_y" value="0.0"/>
-    <!-- <xacro:property name="power_bank_offset_z" value="0.0"/> -->
     <!-- Define colors -->
     <material name="white">

File: description/ros2_control.xacro (robot description, xacro)
@@ -23,12 +23,4 @@
             </joint>
         </ros2_control>
-        <xacro:if value="$(arg ros2_control)">
-            <gazebo>
-                <plugin name="gazebo_ros2_control" filename="libgazebo_ros2_control.so">
-                    <parameters>$(find ks-robo-car)/config/ros2_controllers.yaml</parameters>
-                    <!-- <parameters>$(find ks-robo-car)/config/gaz_ros2_ctl_use_sim.yaml</parameters> -->
-                </plugin>
-            </gazebo>
-        </xacro:if>
     </xacro:if>
     <xacro:unless value="$(arg sim_mode)">
@@ -39,5 +31,5 @@
                 <param name="right_wheel_name">right_wheel_joint</param>
                 <param name="loop_rate">30</param>
-                <param name="device">/dev/ttyUSB0</param>
+                <param name="device">/dev/serial/by-id/usb-1a86_USB_Serial-if00-port0</param>
                 <param name="baud_rate">57600</param>
                 <param name="timeout">1000</param>
@@ -62,3 +54,11 @@
         </ros2_control>
     </xacro:unless>
+    <xacro:if value="$(arg ros2_control)">
+        <gazebo>
+            <plugin name="gazebo_ros2_control" filename="libgazebo_ros2_control.so">
+                <parameters>$(find ks-robo-car)/config/ros2_controllers.yaml</parameters>
+                <parameters>$(find ks-robo-car)/config/ros2_controller_sim_mode.yaml</parameters>
+            </plugin>
+        </gazebo>
+    </xacro:if>
 </robot>
